File: BNC/BNC-V003.sch (EAGLE design)
At the start: 23 parts, among them IC1 LM339N, IC2 74AC08N, J1 POWER_JACKSLT

Commit message: yyyyyyyy enter the commit message for your changes. Lines starting
Parts:
- removed C2: 0.1uF, SparkFun-Capacitors:0.1UF-25V-5%(0603)
- added C3: (no value), SparkFun-Capacitors:0.1UF-50V-20%(PTH)KIT-EZ
- C1: value 0.1uF -> (none); device SparkFun-Capacitors:0.1UF-25V-5%(0603) -> SparkFun-Capacitors:0.1UF-50V-20%(PTH)KIT-EZ
Connections:
- net GND: now also U$11.GND, U$12.GND, U$13.GND, U$14.GND
- net N$11: now also C1.2; no longer C2.2
- net N$7: now also C3.2; no longer C1.2
- net N$8: now also C3.1; no longer C1.1
- net N$9: now also C1.1; no longer C2.1
Other:
- moved on the sheet: C1
Changed lines of the file:
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@@
 <part name="SUPPLY5" library="SparkFun-Aesthetics" deviceset="5V" device=""/>
 <part name="R5" library="SparkFun-Resistors" deviceset="10KOHM-1/4W-1%(PTH)" device="HORIZ" value="10k"/>
-<part name="C1" library="SparkFun-Capacitors" deviceset="0.1UF-25V-5%(0603)" device="" value="0.1uF"/>
-<part name="C2" library="SparkFun-Capacitors" deviceset="0.1UF-25V-5%(0603)" device="" value="0.1uF"/>
 <part name="IAG3-D3" library="SparkFun-LED" deviceset="LTE-302" device=""/>
 <part name="GND6" library="SparkFun-Aesthetics" deviceset="GND" device=""/>
@@
 <part name="SUPPLY6" library="SparkFun-Aesthetics" deviceset="5V" device=""/>
 <part name="GND3" library="SparkFun-Aesthetics" deviceset="GND" device=""/>
+<part name="GND4" library="SparkFun-Aesthetics" deviceset="GND" device=""/>
+<part name="GND5" library="SparkFun-Aesthetics" deviceset="GND" device=""/>
+<part name="GND10" library="SparkFun-Aesthetics" deviceset="GND" device=""/>
+<part name="GND11" library="SparkFun-Aesthetics" deviceset="GND" device=""/>
+<part name="C3" library="SparkFun-Capacitors" deviceset="0.1UF-50V-20%(PTH)" device="KIT-EZ"/>
+<part name="C1" library="SparkFun-Capacitors" deviceset="0.1UF-50V-20%(PTH)" device="KIT-EZ"/>
 </parts>
 <sheets>
@@
 <instance part="SUPPLY5" gate="G$1" x="43.18" y="-22.86"/>
 <instance part="R5" gate="G$1" x="50.8" y="-25.4"/>
-<instance part="C1" gate="G$1" x="7.62" y="63.5"/>
-<instance part="C2" gate="G$1" x="10.16" y="-17.78"/>
 <instance part="IAG3-D3" gate="G$1" x="193.04" y="20.32" rot="R270"/>
 <instance part="GND6" gate="1" x="177.8" y="15.24"/>
@@
 <instance part="SUPPLY6" gate="G$1" x="101.6" y="48.26"/>
 <instance part="GND3" gate="1" x="101.6" y="30.48"/>
+<instance part="GND4" gate="1" x="220.98" y="35.56"/>
+<instance part="GND5" gate="1" x="223.52" y="-12.7"/>
+<instance part="GND10" gate="1" x="152.4" y="-12.7"/>
+<instance part="GND11" gate="1" x="152.4" y="40.64"/>
+<instance part="C3" gate="G$1" x="2.54" y="63.5"/>
+<instance part="C1" gate="G$1" x="5.08" y="-17.78"/>
 </instances>
 <busses>
@@
 <pinref part="IC2" gate="P" pin="GND"/>
 <pinref part="GND3" gate="1" pin="GND"/>
+</segment>
+<segment>
+<pinref part="U$11" gate="G$1" pin="GND"/>
+<pinref part="GND11" gate="1" pin="GND"/>
+<wire x1="144.78" y1="45.72" x2="152.4" y2="45.72" width="0.1524" layer="91"/>
+<wire x1="152.4" y1="45.72" x2="152.4" y2="43.18" width="0.1524" layer="91"/>
+</segment>
+<segment>
+<pinref part="U$12" gate="G$1" pin="GND"/>
+<pinref part="GND10" gate="1" pin="GND"/>
+<wire x1="144.78" y1="-7.62" x2="152.4" y2="-7.62" width="0.1524" layer="91"/>
+<wire x1="152.4" y1="-7.62" x2="152.4" y2="-10.16" width="0.1524" layer="91"/>
+</segment>
+<segment>
+<pinref part="U$14" gate="G$1" pin="GND"/>
+<pinref part="GND5" gate="1" pin="GND"/>
+<wire x1="215.9" y1="-10.16" x2="223.52" y2="-10.16" width="0.1524" layer="91"/>
+</segment>
+<segment>
+<pinref part="U$13" gate="G$1" pin="GND"/>
+<pinref part="GND4" gate="1" pin="GND"/>
+<wire x1="213.36" y1="40.64" x2="220.98" y2="40.64" width="0.1524" layer="91"/>
+<wire x1="220.98" y1="40.64" x2="220.98" y2="38.1" width="0.1524" layer="91"/>
 </segment>
 </net>
@@
 <pinref part="COS" gate="G$1" pin="GND"/>
 <wire x1="-7.62" y1="63.5" x2="-7.62" y2="60.96" width="0.1524" layer="91"/>
-<pinref part="C1" gate="G$1" pin="2"/>
-<wire x1="-7.62" y1="60.96" x2="7.62" y2="60.96" width="0.1524" layer="91"/>
-<wire x1="7.62" y1="60.96" x2="12.7" y2="60.96" width="0.1524" layer="91"/>
+<wire x1="-7.62" y1="60.96" x2="2.54" y2="60.96" width="0.1524" layer="91"/>
+<wire x1="2.54" y1="60.96" x2="12.7" y2="60.96" width="0.1524" layer="91"/>
 <wire x1="12.7" y1="60.96" x2="12.7" y2="40.64" width="0.1524" layer="91"/>
-<junction x="7.62" y="60.96"/>
 <wire x1="12.7" y1="40.64" x2="33.02" y2="40.64" width="0.1524" layer="91"/>
 <wire x1="33.02" y1="40.64" x2="38.1" y2="40.64" width="0.1524" layer="91"/>
@@
 <pinref part="IC1" gate="A" pin="+IN"/>
 <pinref part="IC1" gate="B" pin="-IN"/>
+<pinref part="C3" gate="G$1" pin="2"/>
+<junction x="2.54" y="60.96"/>
 </segment>
 </net>
@@
 <segment>
 <pinref part="COS" gate="G$1" pin="OUT"/>
-<pinref part="C1" gate="G$1" pin="1"/>
-<wire x1="-2.54" y1="68.58" x2="7.62" y2="68.58" width="0.1524" layer="91"/>
-<wire x1="7.62" y1="68.58" x2="15.24" y2="68.58" width="0.1524" layer="91"/>
+<wire x1="-2.54" y1="68.58" x2="2.54" y2="68.58" width="0.1524" layer="91"/>
+<wire x1="2.54" y1="68.58" x2="15.24" y2="68.58" width="0.1524" layer="91"/>
 <wire x1="15.24" y1="68.58" x2="15.24" y2="76.2" width="0.1524" layer="91"/>
-<junction x="7.62" y="68.58"/>
 <wire x1="15.24" y1="76.2" x2="38.1" y2="76.2" width="0.1524" layer="91"/>
 <wire x1="15.24" y1="68.58" x2="22.86" y2="68.58" width="0.1524" layer="91"/>
@@
 <pinref part="IC1" gate="A" pin="-IN"/>
 <pinref part="IC1" gate="B" pin="+IN"/>
+<pinref part="C3" gate="G$1" pin="1"/>
+<junction x="2.54" y="68.58"/>
 </segment>
 </net>
@@
 <segment>
 <pinref part="SIN" gate="G$1" pin="OUT"/>
-<pinref part="C2" gate="G$1" pin="1"/>
-<wire x1="0" y1="-12.7" x2="10.16" y2="-12.7" width="0.1524" layer="91"/>
-<wire x1="10.16" y1="-12.7" x2="27.94" y2="-12.7" width="0.1524" layer="91"/>
+<wire x1="0" y1="-12.7" x2="5.08" y2="-12.7" width="0.1524" layer="91"/>
+<wire x1="5.08" y1="-12.7" x2="27.94" y2="-12.7" width="0.1524" layer="91"/>
 <wire x1="27.94" y1="-12.7" x2="27.94" y2="-2.54" width="0.1524" layer="91"/>
-<junction x="10.16" y="-12.7"/>
 <wire x1="27.94" y1="-2.54" x2="38.1" y2="-2.54" width="0.1524" layer="91"/>
 <wire x1="27.94" y1="-12.7" x2="27.94" y2="-33.02" width="0.1524" layer="91"/>
@@
 <pinref part="IC1" gate="C" pin="-IN"/>
 <pinref part="IC1" gate="D" pin="+IN"/>
+<pinref part="C1" gate="G$1" pin="1"/>
+<junction x="5.08" y="-12.7"/>
 </segment>
 </net>
@@
 <pinref part="SIN" gate="G$1" pin="GND"/>
 <wire x1="-5.08" y1="-17.78" x2="-5.08" y2="-20.32" width="0.1524" layer="91"/>
-<pinref part="C2" gate="G$1" pin="2"/>
-<wire x1="-5.08" y1="-20.32" x2="10.16" y2="-20.32" width="0.1524" layer="91"/>
+<wire x1="-5.08" y1="-20.32" x2="5.08" y2="-20.32" width="0.1524" layer="91"/>
+<wire x1="5.08" y1="-20.32" x2="10.16" y2="-20.32" width="0.1524" layer="91"/>
 <wire x1="10.16" y1="-20.32" x2="10.16" y2="-38.1" width="0.1524" layer="91"/>
 <junction x="10.16" y="-20.32"/>
@@
 <pinref part="IC1" gate="C" pin="+IN"/>
 <pinref part="IC1" gate="D" pin="-IN"/>
-</segment>
-</net>
+<pinref part="C1" gate="G$1" pin="2"/>
+<junction x="5.08" y="-20.32"/>
+</segment>
+</net>
